File: corne-wireless-chocolate/pcb/corne-wireless-chocolate.kicad_pcb (KiCad board)
At the start: 2 copper layers, 275.5 x 105.6 mm, 132 parts, among them J2 OLED, J5 Breakaway_Tabs, J7 OLED, SW1 SW_PUSH, SW10 SW_PUSH, SW11 SW_PUSH, SW12 SW_PUSH, SW13 SW_PUSH, SW14 SW_PUSH, SW15 SW_PUSH, SW16 SW_PUSH, SW17 SW_PUSH, SW18 SW_PUSH, SW19 SW_PUSH, SW2 SW_PUSH, SW20 SW_PUSH, SW21 SW_PUSH, SW22 SW_PUSH, SW23 SW_PUSH, SW24 SW_PUSH, SW25 SW_PUSH, SW26 SW_PUSH, SW27 SW_PUSH, SW28 SW_PUSH, SW29 SW_PUSH, SW3 SW_PUSH, SW30 SW_PUSH, SW31 SW_PUSH, SW32 SW_PUSH, SW33 SW_PUSH, SW34 SW_PUSH, SW35 SW_PUSH, SW36 SW_PUSH, SW37 SW_PUSH, SW38 SW_PUSH, SW39 SW_PUSH, SW4 SW_PUSH, SW40 SW_PUSH, SW41 SW_PUSH, SW42 SW_PUSH, SW5 SW_PUSH, SW6 SW_PUSH, SW7 SW_PUSH, SW8 SW_PUSH, SW9 SW_PUSH, U1 ProMicro, U2 ProMicro

Commit message: feat: add the support for 3x5
Parts:
- removed the Ref** at (50.7, 74.4)
- moved D14 18.0 mm to (49.7, 88.4)
- moved D2 15.3 mm to (43.2, 54.4), turned to 180 degrees
- moved D8 15.1 mm to (43.2, 73.4), turned to 180 degrees
- moved D22 14.9 mm to (280.2, 54.4), turned to 180 degrees
- moved D28 14.9 mm to (280.2, 73.4), turned to 180 degrees
- moved D34 11.0 mm to (280.2, 75.4), turned to 180 degrees
- turned SW14 to 0 degrees
- turned SW2 to 0 degrees
- turned SW22 to 90 degrees
- turned SW28 to 90 degrees
- turned SW34 to 90 degrees
- turned SW8 to 0 degrees
Routing:
- net row2_r: track 145.0 -> 172.7 mm
- net row1_r: track 136.8 -> 152.7 mm
- net Net-(D28-Pad2): track 10.9 -> 25.7 mm
- net Net-(D22-Pad2): track 10.9 -> 25.7 mm
- net row0_r: track 135.6 -> 150.1 mm
- net Net-(D8-Pad2): track 10.6 -> 22.8 mm
- net Net-(D2-Pad2): track 10.8 -> 20.0 mm
- net Net-(D34-Pad2): track 10.8 -> 2.34 mm, vias 1 -> 0
- net col0_r: track 183.7 -> 176.3 mm
- net row0: track 149.3 -> 156.3 mm
- net col1: track 138.8 -> 145.2 mm, vias 4 -> 5
- net row1: track 147.6 -> 153.8 mm, vias 0 -> 1
- net Net-(D14-Pad2): track 10.5 -> 5.34 mm, vias 1 -> 0
- net row2: track 148.5 -> 151.8 mm
- net col0: track 168.4 -> 167.4 mm
Other:
- outline, holes or cut-outs redrawn
